File: smart-filament-drybox-monitor.kicad_sch (KiCad schematic)
At the start: 39 parts, among them J2 Conn_01x06, J3 USB_C_Receptacle_USB2.0_14P, P4 AFC07-S24FCC-00, Q3 AO3400A, SW1 SW_Push, SW2 SW_Push, U1 ESP32-C6-MINI-1/U, U2 SHT4x

Commit message: added a title for the usb c power section
Other:
- note added: "USB-C & Power"
Changed lines of the file:
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@@
 	(generator_version "9.0")
 	(paper "A4")
+	(text "USB-C & Power\n"
+		(exclude_from_sim no)
+		(at 21.082 15.24 0)
+		(effects
+			(font
+				(size 1.27 1.27)
+			)
+		)
+	)
 	(text "EN & RESET Buttons"
 		(exclude_from_sim no)
